Commit message: 修改了模型底盘位置和机器人配色

File: urdf/robot/openarmx_robot.urdf (robot description, URDF)
Before this commit: robot openarmx, 30 links, 29 joints
Links:
- link openarmx_body_link0: geometry collision mesh filename=package://openarmx_description/meshes/body/v10/collision/bo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 scale=1.0 1.0 1.0; visual mesh filename=package://openarmx_description/meshes/body/v10/visual/body_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 scale=1.0 1.0 1.0
Joints:
- joint openarmx_left_openarmx_body_link0_joint: origin xyz=0.0 0.031 0.698 rpy=-1.5708 0 0 -> xyz=0.0 0.031 0.735 rpy=-1.5708 0 0
- joint openarmx_right_openarmx_body_link0_joint: origin xyz=0.0 -0.031 0.698 rpy=1.5708 0 0 -> xyz=0.0 -0.031 0.735 rpy=1.5708 0 0

File: urdf/robot/v10.urdf.xacro (robot description, xacro)
@@ -22,7 +22,11 @@
   <xacro:arg name="fake_sensor_commands" default="false" />
   <xacro:arg name="bimanual" default="false" />
-  <xacro:arg name="right_arm_base_xyz" default="0.0 -0.031 0.698" />
+  <!-- <xacro:arg name="right_arm_base_xyz" default="0.0 -0.031 0.698" />
   <xacro:arg name="right_arm_base_rpy" default="1.5708 0 0" />
   <xacro:arg name="left_arm_base_xyz" default="0.0 0.031 0.698" />
+  <xacro:arg name="left_arm_base_rpy" default="-1.5708 0 0" /> -->
+  <xacro:arg name="right_arm_base_xyz" default="0.0 -0.031 0.735" />
+  <xacro:arg name="right_arm_base_rpy" default="1.5708 0 0" />
+  <xacro:arg name="left_arm_base_xyz" default="0.0 0.031 0.735" />
   <xacro:arg name="left_arm_base_rpy" default="-1.5708 0 0" />
   <xacro:arg name="can_fd" default="false" />
