Commit message: 修复了错误的机器人模型

File: urdf/body/openarmx_body_macro.xacro (robot description, xacro)
@@ -23,5 +23,5 @@
         <xacro:openarmx-body-kinematics config="${kinematics_link}" name="${name}" />
         <geometry>
-          <mesh filename="package://${description_pkg}/meshes/body/${body_type}/visual/${name}.dae" scale="0.001 0.001 0.001" />
+          <mesh filename="package://${description_pkg}/meshes/body/${body_type}/visual/${name}.dae" scale="1.0 1.0 1.0" />
         </geometry>
       </visual>
@@ -29,5 +29,5 @@
         <xacro:openarmx-body-kinematics config="${kinematics_link}" name="${name}" />
         <geometry>
-          <mesh filename="package://openarmx_description/meshes/body/${body_type}/collision/${name}_symp.stl" scale="0.001 0.001 0.001" />
+          <mesh filename="package://openarmx_description/meshes/body/${body_type}/collision/${name}_symp.stl" scale="1.0 1.0 1.0" />
           <!-- <mesh filename="package://openarmx_description/meshes/arm/${arm_type}/collision/${name}.stl" scale="0.001 0.001 0.001" /> -->
         </geometry>

Commit message: 修复了模型在urdf viewer里显示错误

File: urdf/body/openarmx_body_macro.xacro (robot description, xacro)
@@ -29,6 +29,5 @@
         <xacro:openarmx-body-kinematics config="${kinematics_link}" name="${name}" />
         <geometry>
-          <mesh filename="package://openarmx_description/meshes/body/${body_type}/collision/${name}_symp.stl" scale="1.0 1.0 1.0" />
-          <!-- <mesh filename="package://openarmx_description/meshes/arm/${arm_type}/collision/${name}.stl" scale="0.001 0.001 0.001" /> -->
+          <mesh filename="package://openarmx_description/meshes/body/${body_type}/collision/${name}_symp.stl" scale="0.001 0.001 0.001" />
         </geometry>
       </collision>

File: urdf/robot/openarmx_robot.urdf (robot description, URDF)
Before this commit: robot openarmx, 30 links, 29 joints
Links:
- link openarmx_body_link0: geometry collision mesh filename=package://openarmx_description/meshes/body/v10/collision/bo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 scale=0.001 0.001 0.001; visual mesh filename=package://openarmx_description/meshes/body/v10/visual/body_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 scale=1.0 1.0 1.0
